Commit message: launch file is fixed and lidar is added

File: src/urdf/quadrotor.urdf (robot description, URDF)
Before this commit: robot hector_quadrotor, 1 links, 0 joints
Links:
- added link lidar_link
Joints:
- added joint lidar_joint: type fixed, parent base_link, child lidar_link, origin xyz=0.1 0 0.05 rpy=0 0 0
